File: PCB/Macropad.kicad_pcb (KiCad board)
At the start: 2 copper layers, 74.1 x 64.6 mm, 20 parts, among them SW1 RotaryEncoder_Switch_MP, SW10 SW_Push, SW13 SW_Push, SW14 SW_Push, SW5 SW_Push, SW6 SW_Push, SW9 SW_Push, U1 XIAO-RP2040-DIP

Commit message: Fixed version of the PCB
Parts:
- added D13: SK6812, LED_SMD:LED_SK6812_PLCC4_5.0x5.0mm_P3.2mm, F.Cu at (3.56, 2.81)
- D1: value SK6812MINI -> SK6812
- moved D4 0.10 mm to (171.5, 62.0)
Connections:
- D1 pad 1: Net-(D1-DOUT) -> GND
- D1 pad 2: GND -> LEDs
- D1 pad 3: LEDs -> +5V
- D1 pad 4: +5V -> Net-(D1-VDD)
- D2 pad 3: Net-(D1-DOUT) -> Net-(D1-VDD)
Routing:
- net GND: track 76.5 -> 129.2 mm
- net Net-(D1-VDD): track 0.00 -> 20.7 mm
- net Net-(D1-DOUT): track 16.3 -> 0.00 mm
- net +5V: track 173.0 -> 177.4 mm
- net LEDs: track 6.53 -> 4.21 mm
